File: KiCAD/usb-lab-bench-psu/power_lm5176.kicad_sch (KiCad schematic)
At the start: 49 parts, among them Q4 NMOS, Q5 DMN6040SK3, Q6 DMN6040SK3, Q7 DMN6040SK3, Q8 DMN6040SK3, U17 LM5176PWP

Commit message: Fixed label directions
Changed lines of the file:
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@@
 	)
 	(hierarchical_label "VIN"
-		(shape output)
+		(shape input)
 		(at 30.48 25.4 180)
 		(effects
@@
 	)
 	(hierarchical_label "FB"
-		(shape output)
+		(shape input)
 		(at 101.6 88.9 0)
 		(effects
@@
 	)
 	(hierarchical_label "VOUT"
-		(shape input)
+		(shape output)
 		(at 275.59 35.56 0)
 		(effects
@@
 	)
 	(hierarchical_label "~{EN}"
-		(shape output)
+		(shape input)
 		(at 24.13 180.34 180)
 		(effects
@@
 	)
 	(hierarchical_label "VIN"
-		(shape output)
+		(shape input)
 		(at 52.07 152.4 90)
 		(effects
