File: KiCAD/usb-lab-bench-psu/usb-lab-bench-psu.kicad_sch (KiCad schematic)
At the start: 12 parts, among them J1 Conn_02x02_Top_Bottom, J10 Conn_01x04, J11 Conn_01x04, J12 Conn_01x02, J2 Conn_01x04, J3 Conn_01x04, J4 Conn_01x02, J5 Conn_01x02, J6 Conn_01x04, J7 Conn_01x04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

Commit message: tweaked design of current limiter, added GPIO expander to USB-PD circuit
Connections:
- net USB-PD/ALERT is gone; now on net USB_PD_GND: J2.3 (Pin_3)
- net HOST-USB-RESET: now also J3.1 (Pin_1)
- net HOST_GND: now also J3.3 (Pin_3)
- net HOST-USB_~{INT}: now reaches J3.2 (Pin_2)
- net USB-PD/ATTACH renamed USB-PD/~{INT}
Other:
- sheet Host ports: added USB_~{INT}; removed USB_ALERT, USB_ATTACH
- sheet IO-Board ports: added 3V3; removed +3V3
- sheet USB-PD ports: added ~{INT}; removed ALERT, ATTACH
